Commit message: working-ish

File: src/follow_me/urdf/tracer_mini.urdf (robot description, URDF)
Before this commit: robot tracer_mini, 9 links, 8 joints
Links:
- link base_link: geometry collision mesh filename=file://$(find follow_me)/meshes/base_link.STL; visual mesh filename=file://$(find follow_me)/meshes/base_link.STL
- link camera_link: geometry collision mesh filename=file://$(find follow_me)/meshes/camera_Link.STL; visual mesh filename=file://$(find follow_me)/meshes/camera_Link.STL
- link laser_Link: geometry collision mesh filename=file://$(find follow_me)/meshes/laser_Link.STL; visual mesh filename=file://$(find follow_me)/meshes/laser_Link.STL
